File: cad/elec/arduino-micro-dmx.kicad_pcb (KiCad board)
At the start: 2 copper layers, 74.9 x 55.2 mm, 31 parts, among them CON1 BARREL_JACK, P2 DMX IN, P3 DMX OUT, P4 I2C OUT, SW1 TERM_SELECTOR, U1 ROE-0505S, U2 ARDUINO_MICRO, U3 ADuM1286, U4 MAX488E

Commit message: Polishing
Connections:
- U2 pad 3: /DMX_IN -> /DMX_OUT
- U2 pad 4: /DMX_OUT -> /DMX_IN
- U3 pad 2: /DMX_OUT -> /DMX_IN
- U3 pad 3: /DMX_IN -> /DMX_OUT
Routing:
- net GNDA: track 146.3 -> 182.7 mm, vias 17 -> 13
- net GND: track 393.6 -> 405.8 mm, vias 33 -> 32
- net /DMX_OUT: track 13.7 -> 20.5 mm
- net /DMX_IN: track 20.5 -> 13.7 mm
- net Net-(R2-Pad2): track 6.20 -> 9.87 mm
- net /DMX_IN_B: track 60.9 -> 60.0 mm
Other:
- net class Default: via_dia 0.9 -> 1.6; via_drill 0.5 -> 0.8
- board text added: "This documentation describes Open Hardware and is licensed under the CERN OHL v. 1.2. You may redistribute and modify this documentation under the terms of the CERN OHL v.1.2. (http://ohwr.org/cernohl). This documentation is distributed WITHOUT ANY EXPRESS OR IMPLIED WARRANTY, INCLUDING OF MERCHANTABILITY, SATISFACTORY QUALITY AND FITNESS FOR A PARTICULAR PURPOSE. Please see the CERN OHL v.1.2 fo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"
